File: EEPROM_PROGRAMER_V3.0/EEPROM_PROGRAMER_V3.0.kicad_pcb (KiCad board)
At the start: 2 copper layers, 8 parts

Commit message: Some changes at the V3.0 design
Parts:
- added EEPROM SOCKET: DIP_Socket-28_W11.9_W12.7_W15.24_W17.78_W18.5_3M_228-1277-0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, Socket:DIP_Socket-28_W11.9_W12.7_W15.24_W17.78_W18.5_3M_228-1277-00-0602J, F.Cu at (133.6, 127.6)
- added REF**: SW_08xDIP, Button_Switch_SMD:SW_DIP_SPSTx08_Slide_6.7x21.88mm_W8.61mm_P2.54mm_LowProfile, F.Cu at (171.3, 70.6)
- added U1: 74HC595, Package_SO:SOIC-16_3.9x9.9mm_P1.27mm, F.Cu at (146.9, 136.5)
- added U1: 74HC595, Package_SO:SOIC-16_3.9x9.9mm_P1.27mm, F.Cu at (144.5, 102.2)

Commit message: V3.0 is ready to order
Parts:
- removed 74HC595 (x2): DIP-16_W7.62mm_Socket_LongPads, Package_DIP:DIP-16_W7.62mm_Socket_LongPads
- removed EEPROM SOCKET: DIP_Socket-28_W11.9_W12.7_W15.24_W17.78_W18.5_3M_228-1277-0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, Socket:DIP_Socket-28_W11.9_W12.7_W15.24_W17.78_W18.5_3M_228-1277-00-0602J
- removed the REF** at (230.8, 132.5)
- removed the REF** at (202.7, 138.2)
- removed the REF** at (171.3, 70.6)
- removed the REF** at (230.9, 135.5)
- removed the U1 at (144.5, 102.2)
- added +: PinSocket_1x02_P2.54mm_Vertical, Connector_PinSocket_2.54mm:PinSocket_1x02_P2.54mm_Vertical, F.Cu at (176.1, 128.0)
- added +: PinSocket_1x02_P2.54mm_Vertical, Connector_PinSocket_2.54mm:PinSocket_1x02_P2.54mm_Vertical, F.Cu at (176.1, 102.3)
- added REF**: EN, LED_SMD:LED_0805_2012Metric_Pad1.15x1.40mm_HandSolder, F.Cu at (124.2, 130.6)
- added REF**: SW_DIP_SPSTx04_Slide_9.78x12.34mm_W8.61mm_P2.54mm, Button_Switch_SMD:SW_DIP_SPSTx04_Slide_9.78x12.34mm_W8.61mm_P2.54mm, F.Cu at (133.0, 134.6)
- added REF**: R_0603_1608Metric_Pad0.98x0.95mm_HandSolder, Resistor_SMD:R_0603_1608Metric_Pad0.98x0.95mm_HandSolder, F.Cu at (124.2, 132.6)
- added REF**11: R_0603_1608Metric_Pad0.98x0.95mm_HandSolder, Resistor_SMD:R_0603_1608Metric_Pad0.98x0.95mm_HandSolder, F.Cu at (131.2, 142.7)
- added REF**12: R_0603_1608Metric_Pad0.98x0.95mm_HandSolder, Resistor_SMD:R_0603_1608Metric_Pad0.98x0.95mm_HandSolder, F.Cu at (133.2, 142.7)
- added REF**13: R_0603_1608Metric_Pad0.98x0.95mm_HandSolder, Resistor_SMD:R_0603_1608Metric_Pad0.98x0.95mm_HandSolder, F.Cu at (135.2, 142.7)
- added REF**14: R_0603_1608Metric_Pad0.98x0.95mm_HandSolder, Resistor_SMD:R_0603_1608Metric_Pad0.98x0.95mm_HandSolder, F.Cu at (137.2, 142.7)
- added U5: 74HC595, Package_SO:SOIC-16_3.9x9.9mm_P1.27mm, F.Cu at (145.9, 132.7)
- U2: renamed from EEPROM SOCKET; value DIP_Socket-28_W11.9_W12.7_W15.24_W17.78_W18.5_3M_228-1277-00-0602J -> EEPROM SOCKET
- moved G*** 64.8 mm to (169.6, 135.2), turned to 0 degrees
- moved U1 11.0 mm to (157.3, 132.7), turned to -90 degrees
- moved U2 5.02 mm to (133.5, 122.5)
Routing:
- net (no net): track 918.8 -> 1497.0 mm, vias 13 -> 24
Other:
- board outline added: 58.9 x 53.3 mm
- board text added: "DATA"
- board text added: "EN"
- board text added: "OE"
- board text added: "SW1"
- board text added: "SW2"
- board text added: "SW3"
- board text added: "V3.0"
- board text removed: "DATA_IN"
- board text removed: "NO"
- board text removed: "V2.0"
