File: EEPROM_PROGRAMER_V3.0/EEPROM_PROGRAMER_V3.0.kicad_sch (KiCad schematic)
At the start: 1 part, among them U1 74HC595

Commit message: V3.0 is ready to order
Parts:
- added 1K?: 1K, symbol Device:R
- added D?: LED, symbol Device:LED
- added U2: 28C256, symbol Memory_EEPROM:28C256
- added U5: 74HC595, Package_SO:SOIC-16_3.9x9.9mm_P1.27mm, symbol 74xx:74HC595
Connections:
- net at U1.1 (QB): now also U2.9 (A1)
- net VCC: now reaches U1.10 (~{SRCLR})
- net VCC: now also U1.16 (VCC), D?.2 (A), U2.28 (VCC), U5.10 (~{SRCLR}), U5.16 (VCC)
- net CLK: now reaches U1.11 (SRCLK)
- net CLK: now also U5.11 (SRCLK)
- net RCLK: now reaches U1.12 (RCLK)
- net RCLK: now also U5.12 (RCLK)
- net ~{OE}: now reaches U1.13 (~{OE})
- net ~{OE}: now also U5.13 (~{OE})
- net DATA: now reaches U1.14 (SER)
- net at U1.15 (QA): now also U2.10 (A0)
- net at U1.2 (QC): now also U2.8 (A2)
- net at U1.3 (QD): now also U2.7 (A3)
- net at U1.4 (QE): now also U2.6 (A4)
- net at U1.5 (QF): now also U2.5 (A5)
- net at U1.6 (QG): now also U2.4 (A6)
- net at U1.7 (QH): now also U2.3 (A7)
- net Earth: now reaches U1.8 (GND)
- net Earth: now also 1K?.1, U2.14 (GND), U5.8 (GND)
- net at U1.9 (QH'): now also U5.14 (SER)
- new net: U2.24 (A9), U5.1 (QB)
- new net: U2.25 (A8), U5.15 (QA)
- new net: U2.21 (A10), U5.2 (QC)
- new net: U2.23 (A11), U5.3 (QD)
- new net: U2.2 (A12), U5.4 (QE)
- new net: U2.26 (A13), U5.5 (QF)
- new net: U2.1 (A14), U5.6 (QG)
- new net: 1K?.2, D?.1 (K)
- no-connect marks 0 -> 2
Other:
- moved on the sheet: U1
